Commit message: final

File: urdf/robodog.urdf (robot description, URDF)
Before this commit: robot robodog, 19 links, 18 joints
Links:
- added link camera_link
- added link kinect_link, mass 0.1; collision box size=0.00 0.00 0.00; visual box size=0.02 0.08 0.02
- link base_link: geometry collision box size=0.4 0.25 0.05; visual box size=0.4 0.25 0.05
- link imu_link: geometry collision cylinder length=0.01 radius=0.2; visual cylinder length=0.01 radius=0.01
- link lidar_link: mass 0.5 -> 0.1
Joints:
- added joint kinect_base: type fixed, parent base_link, child kinect_link, origin xyz=0.20 0.0 0.01 rpy=0.0 0.0 0.0
- added joint kinect_camera: type fixed, parent kinect_link, child camera_link, origin xyz=0.00 0.0 0.000 rpy=-1.57 0.0 -1.57
- joint base_leg_bl: origin xyz=-0.13 0.13 0.245 rpy=0.0 1.57 0.0 -> xyz=-0.13 0.13 -0.005 rpy=0.0 1.57 0.0
- joint base_leg_br: origin xyz=-0.13 -0.13 0.245 rpy=0.0 1.57 0.0 -> xyz=-0.13 -0.13 -0.005 rpy=0.0 1.57 0.0
- joint base_leg_fl: origin xyz=0.13 0.13 0.245 rpy=0.0 1.57 0.0 -> xyz=0.13 0.13 -0.005 rpy=0.0 1.57 0.0
- joint base_leg_fr: origin xyz=0.13 -0.13 0.245 rpy=0.0 1.57 0.0 -> xyz=0.13 -0.13 -0.005 rpy=0.0 1.57 0.0
- joint imu_base: origin xyz=0.0 0.0 0.00 rpy=0.0 0.0 0.0 -> xyz=0.0 0.0 0.0 rpy=0.0 0.0 0.0
- joint lidar_base: origin xyz=0.14 0.0 0.04 rpy=0.0 0.0 0.0 -> xyz=0.14 0.0 0.055 rpy=0.0 0.0 3.14
